File: board/board.kicad_pcb (KiCad board)
At the start: 2 copper layers, 21 x 13 mm, 1 part

Commit message: initial
Parts:
- added C1: 100nF, Capacitor_SMD:C_0603_1608Metric, F.Cu at (147.6, 96.1)
- added J1: 001_I2C, on_edge:on_edge_2x05_device, F.Cu at (140.0, 96.5)
- added J2: 001_I2C, on_edge:on_edge_2x05_host, F.Cu at (161.0, 96.5)
- added R1: 0R, Resistor_SMD:R_0603_1608Metric, F.Cu at (146.1, 96.3)
- added R2: 0R, Resistor_SMD:R_0603_1608Metric, F.Cu at (154.5, 97.3)
- added R3: 0R, Resistor_SMD:R_0603_1608Metric, F.Cu at (154.4, 100.0)
- added R4: d.n.p, Resistor_SMD:R_0603_1608Metric, F.Cu at (151.0, 101.5)
- added R5: 0R, Resistor_SMD:R_0603_1608Metric, F.Cu at (148.0, 101.5)
- added R6: d.n.p, Resistor_SMD:R_0603_1608Metric, F.Cu at (151.0, 98.5)
- added R7: 0R, Resistor_SMD:R_0603_1608Metric, F.Cu at (148.0, 98.5)
- added R8: d.n.p, Resistor_SMD:R_0603_1608Metric, F.Cu at (151.0, 100.0)
- added R9: 0R, Resistor_SMD:R_0603_1608Metric, F.Cu at (148.0, 100.0)
- added U1: MCP9844x-xMN, Package_DFN_QFN:DFN-8-1EP_3x2mm_P0.5mm_EP1.36x1.46mm, F.Cu at (149.6, 95.4)
- LOGO1: moved to B.Cu
- turned LOGO1 to 180 degrees
Routing:
- net GND: track 0.00 -> 30.9 mm, vias 0 -> 2
- net /temperature/VDD: track 0.00 -> 28.3 mm, vias 0 -> 3
- net /temperature/SCL: track 0.00 -> 21.2 mm, vias 0 -> 2
- net /temperature/SDA: track 0.00 -> 18.6 mm
- net Net-(J1-Pad8): track 0.00 -> 17.0 mm
- net Net-(J1-Pad10): track 0.00 -> 16.2 mm
- net Net-(J1-Pad5): track 0.00 -> 14.8 mm, vias 0 -> 2
- net Net-(J1-Pad4): track 0.00 -> 12.0 mm, vias 0 -> 2
- net Net-(R4-Pad1): track 0.00 -> 6.89 mm
- net Net-(R8-Pad1): track 0.00 -> 5.35 mm
- net /temperature/INT: track 0.00 -> 4.95 mm
- net Net-(J2-Pad4): track 0.00 -> 3.85 mm
- net Net-(J2-Pad5): track 0.00 -> 3.51 mm
- net Net-(R6-Pad1): track 0.00 -> 3.15 mm
Other:
- outline, holes or cut-outs redrawn
