File: board/board.kicad_sch (KiCad schematic)
At the start: 1 part

Commit message: initial
Parts:
- added J1: 001_I2C, on_edge:on_edge_2x05_device, symbol put_on_edge:001_I2C
- added J2: 001_I2C, on_edge:on_edge_2x05_host, symbol put_on_edge:001_I2C
- added R1, R2, R3: 0R, Resistor_SMD:R_0603_1608Metric, symbol Device:R_Small
Connections:
- new net: J1.10 (5V), J2.10 (5V)
- new net: J2.4 (CS/EN), R2.2
- new net: J2.5 (INT), R3.2
- new net: J1.8 (~{RESET}), J2.8 (~{RESET})
- new net: J1.4 (CS/EN), R2.1
- new net: J1.5 (INT), R1.2, R3.1
- new net GND: J1.1 (GND), J2.1 (GND)
- new net temperature/INT: R1.1
- new net temperature/SCL: J1.3 (SCL), J2.3 (SCL)
- new net temperature/SDA: J1.2 (SDA), J2.2 (SDA)
- new net temperature/VDD: J1.9 (3.3V), J2.9 (3.3V)
Other:
- sheet implementation renamed temperature
- sheet temperature: file implementation.kicad_sch -> temperature.kicad_sch
- sheet temperature ports: added GND, INT, SCL, SDA, VDD; removed none
- note removed: "Input connectors go here"
- note removed: "Output connectors go here"
